File: src/OSI 600D Superboard II Cherry Solder Mask.kicad_pcb (KiCad board)
At the start: 2 copper layers, 301.5 x 367.3 mm, 4 parts

Commit message: Removed solder mask from under IC vias. Added homage to origional creator. Added my logo and handle.
Parts:
- added G***: LOGO, SBCLogo:SBCLogo, F.Cu at (329.9, 36.3)
Other:
- board text added: "Bambleweeny57"
- board text added: "Origional by Grant (Klyball) Added to by Jon (Bambleweeny57)"

Commit message: rotated trandistors
Parts:
- moved ? 5.67 mm to (252.9, 54.3), turned to 90 degrees
- moved ? 5.20 mm to (252.8, 35.4), turned to 90 degrees
Changed lines of the file:
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@@
 	(footprint "clipboard:61e98d75-cfc5-48ac-82d2-a25be53cbd38"
 		(layer "F.Cu")
-		(at 248.750267 58.16 -90)
+		(at 252.91 54.31 90)
 		(property "Reference" ""
 			(at 0 0 90)
@@
 	(footprint "clipboard:61e98d75-cfc5-48ac-82d2-a25be53cbd38"
 		(layer "F.Cu")
-		(at 249.390267 39.280002 -90)
+		(at 252.79 35.35 90)
 		(property "Reference" ""
 			(at 0 0 90)

Commit message: Added Most if not all the silkscreen now
Other:
- board text added: "1"
- board text added: "C10"
- board text added: "C11"
- board text added: "C12"
- board text added: "C13"
- board text added: "C21"
- board text added: "C22"
- board text added: "C23"
- board text added: "C24"
- board text added: "C25"
- board text added: "C26"
- board text added: "C27"
- board text added: "C28"
- board text added: "C29"
- board text added: "C30"
- board text added: "C32"
- board text added: "C33"
- board text added: "C35"
- board text added: "C36"
- board text added: "C37"
- board text added: "C38"
- board text added: "C39"
- board text added: "C40"
- board text added: "C41"
- board text added: "C42"
- board text added: "C43"
- board text added: "C44"
- board text added: "C45"
- board text added: "C46"
- board text added: "C47"
- board text added: "C48"
- board text added: "C49"
- board text added: "C5"
- board text added: "C50"
- board text added: "C51"
- board text added: "C52"
- board text added: "C53"
- board text added: "C54"
- board text added: "C55"
- board text added: "C56"
- board text added: "C58"
- board text added: "C59"
- board text added: "C6"
- board text added: "C60"
- board text added: "C61"
- board text added: "C62"
- board text added: "C63"
- board text added: "C64"
- board text added: "C65"
- board text added: "C66"
- board text added: "C67"
- board text added: "C68"
- board text added: "C69"
- board text added: "C7"
- board text added: "J2"
- board text added: "J3"
- board text added: "R65"
