File: src/OSI 600D Superboard II Cherry Solder Mask.kicad_pcb (KiCad board)
At the start: 2 copper layers, 301.5 x 367.3 mm, 5 parts

Commit message: Finish tenting the vias I wanted to, added the top un populated resistors R38-R49, correct D29 placement, added C8 and C57 I missed.
Other:
- board text added: "C57"
- board text added: "C8"
- board text added: "R38"
- board text added: "R39"
- board text added: "R40"
- board text added: "R41"
- board text added: "R42"
- board text added: "R43"
- board text added: "R44"
- board text added: "R45"
- board text added: "R46"
- board text added: "R47"
- board text added: "R48"
- board text added: "R49"

Commit message: changed name
Other:
- board text added: "Bambelweeny57"
- board text added: "Origional by Grant (Klyball) Added to by Jon (Bambelweeny57)"
- board text removed: "Bambleweeny57"
- board text removed: "Origional by Grant (Klyball) Added to by Jon (Bambleweeny57)"
Changed lines of the file:
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@@
 		)
 	)
-	(gr_text "Origional by Grant (Klyball)\nAdded to by Jon (Bambleweeny57)"
+	(gr_text "Origional by Grant (Klyball)\nAdded to by Jon (Bambelweeny57)"
 		(at 285.69 99.7 0)
 		(layer "F.SilkS")
@@
 		)
 	)
-	(gr_text "Bambleweeny57"
+	(gr_text "Bambelweeny57"
 		(at 352.813 36.1486 0)
 		(layer "F.SilkS")
