File: src/OSI 600D Superboard II Cherry Solder Mask.kicad_pcb (KiCad board)
At the start: 2 copper layers, 301.5 x 367.3 mm, 70 parts, among them SW1 SW_Cherry_MX_1.00u_PCB, SW2 SW_Cherry_MX_1.00u_PCB, U70 DIP-14_W7.62mm_LongPads, U8 DIP-40_W15.24mm_LongPads

Commit message: corrected name
Parts:
- added C11: C_Rect_L10.0mm_W3.0mm_P7.50mm_FKS3_FKP3, Capacitor_THT:C_Rect_L10.0mm_W3.0mm_P7.50mm_FKS3_FKP3, F.Cu at (160.3, 66.2)
- added C33: C_Rect_L10.0mm_W3.0mm_P7.50mm_FKS3_FKP3, Capacitor_THT:C_Rect_L10.0mm_W3.0mm_P7.50mm_FKS3_FKP3, F.Cu at (408.0, 190.4)
- added C52: C_Rect_L10.0mm_W3.0mm_P7.50mm_FKS3_FKP3, Capacitor_THT:C_Rect_L10.0mm_W3.0mm_P7.50mm_FKS3_FKP3, F.Cu at (125.0, 91.6)
- added C55: C_Rect_L10.0mm_W3.0mm_P7.50mm_FKS3_FKP3, Capacitor_THT:C_Rect_L10.0mm_W3.0mm_P7.50mm_FKS3_FKP3, F.Cu at (162.2, 93.9)
- added C7: C_Rect_L10.0mm_W3.0mm_P7.50mm_FKS3_FKP3, Capacitor_THT:C_Rect_L10.0mm_W3.0mm_P7.50mm_FKS3_FKP3, F.Cu at (143.3, 94.4)
- added R57: Potentiometer_Bourns_3266Y_Vertical, Potentiometer_THT:Potentiometer_Bourns_3266Y_Vertical, F.Cu at (153.8, 48.1)
- added R58: Potentiometer_Bourns_3266Y_Vertical, Potentiometer_THT:Potentiometer_Bourns_3266Y_Vertical, F.Cu at (123.7, 73.8)
- added SW2: SW_Cherry_MX_1.00u_PCB, Button_Switch_Keyboard:SW_Cherry_MX_1.00u_PCB, F.Cu at (279.0, 375.8)
- added U41: DIP-24_W15.24mm_LongPads, Package_DIP:DIP-24_W15.24mm_LongPads, F.Cu at (208.5, 145.5)
- moved SW2 0.18 mm to (355.2, 337.7)
- moved SW2 0.18 mm to (336.2, 337.7)
- moved SW2 0.18 mm to (240.9, 337.7)
- moved SW2 0.18 mm to (279.0, 337.7)
- moved SW2 0.18 mm to (412.4, 337.7)
- moved SW2 0.18 mm to (374.3, 337.7)
- moved SW2 0.18 mm to (260.0, 337.7)
- moved SW2 0.18 mm to (393.3, 337.7)
- moved SW2 0.18 mm to (298.1, 337.7)
- moved SW2 0.18 mm to (317.1, 337.7)
Routing:
- net (no net): track 62663.9 -> 62578.8 mm, vias 2555 -> 2510
Other:
- board text added: "Bambelweeny57"
- board text added: "Origional by Grant (Klyball) Added to by Jon (Bambelweeny57)"
- board text removed: "Bambleweeny57"
- board text removed: "C11"
- board text removed: "C33"
- board text removed: "C52"
- board text removed: "C55"
- board text removed: "C7"
- board text removed: "Origional by Grant (Klyball) Added to by Jon (Bambleweeny57)"
- board text removed: "R57"
- board text removed: "R58"
- board text removed: "U41"

Commit message: added key switches
Parts:
- moved SW2 0.13 mm to (355.2, 337.6)
- moved SW2 0.13 mm to (336.2, 337.6)
- moved SW2 0.13 mm to (240.9, 337.6)
- moved SW2 0.13 mm to (221.9, 337.6)
- moved SW2 0.13 mm to (279.0, 337.6)
- moved SW2 0.13 mm to (183.8, 337.6)
- moved SW2 0.13 mm to (412.4, 337.6)
- moved SW2 0.13 mm to (374.3, 337.6)
- moved SW2 0.13 mm to (260.0, 337.6)
- moved SW2 0.13 mm to (393.3, 337.6)
- moved SW2 0.13 mm to (279.0, 375.7)
- moved SW2 0.13 mm to (298.1, 337.6)
- moved SW2 0.13 mm to (317.1, 337.6)
- moved SW2 0.13 mm to (164.7, 337.6)
- moved SW2 0.13 mm to (202.8, 337.6)
Routing:
- net (no net): vias 2510 -> 2261

Commit message: Added J2 and J2 footprints and models
Parts:
- added J2: CONN_SDA-41815_12_RA_MOL, OSI:CONN_SDA-41815_12_RA_MOL, F.Cu at (165.8, 35.8)
- added J3: CONN_SDA-41815_12_RA_MOL, OSI:CONN_SDA-41815_12_RA_MOL, F.Cu at (312.9, 35.8)
- added R38: R_Axial_DIN0207_L6.3mm_D2.5mm_P2.54mm_Vertical, Resistor_THT:R_Axial_DIN0207_L6.3mm_D2.5mm_P2.54mm_Vertical, F.Cu at (210.9, 44.5)
- added R39: R_Axial_DIN0207_L6.3mm_D2.5mm_P2.54mm_Vertical, Resistor_THT:R_Axial_DIN0207_L6.3mm_D2.5mm_P2.54mm_Vertical, F.Cu at (210.9, 37.1)
- added R40: R_Axial_DIN0207_L6.3mm_D2.5mm_P2.54mm_Vertical, Resistor_THT:R_Axial_DIN0207_L6.3mm_D2.5mm_P2.54mm_Vertical, F.Cu at (184.3, 44.5)
- added R41: R_Axial_DIN0207_L6.3mm_D2.5mm_P2.54mm_Vertical, Resistor_THT:R_Axial_DIN0207_L6.3mm_D2.5mm_P2.54mm_Vertical, F.Cu at (207.1, 37.1)
- added R42: R_Axial_DIN0207_L6.3mm_D2.5mm_P2.54mm_Vertical, Resistor_THT:R_Axial_DIN0207_L6.3mm_D2.5mm_P2.54mm_Vertical, F.Cu at (203.3, 44.5)
- added R43: R_Axial_DIN0207_L6.3mm_D2.5mm_P2.54mm_Vertical, Resistor_THT:R_Axial_DIN0207_L6.3mm_D2.5mm_P2.54mm_Vertical, F.Cu at (203.3, 37.1)
- added R44: R_Axial_DIN0207_L6.3mm_D2.5mm_P2.54mm_Vertical, Resistor_THT:R_Axial_DIN0207_L6.3mm_D2.5mm_P2.54mm_Vertical, F.Cu at (191.9, 44.5)
- added R45: R_Axial_DIN0207_L6.3mm_D2.5mm_P2.54mm_Vertical, Resistor_THT:R_Axial_DIN0207_L6.3mm_D2.5mm_P2.54mm_Vertical, F.Cu at (191.9, 37.1)
- added R46: R_Axial_DIN0207_L6.3mm_D2.5mm_P2.54mm_Vertical, Resistor_THT:R_Axial_DIN0207_L6.3mm_D2.5mm_P2.54mm_Vertical, F.Cu at (188.1, 44.5)
- added R47: R_Axial_DIN0207_L6.3mm_D2.5mm_P2.54mm_Vertical, Resistor_THT:R_Axial_DIN0207_L6.3mm_D2.5mm_P2.54mm_Vertical, F.Cu at (188.1, 37.1)
- added R48: R_Axial_DIN0207_L6.3mm_D2.5mm_P2.54mm_Vertical, Resistor_THT:R_Axial_DIN0207_L6.3mm_D2.5mm_P2.54mm_Vertical, F.Cu at (207.1, 44.5)
- added R49: R_Axial_DIN0207_L6.3mm_D2.5mm_P2.54mm_Vertical, Resistor_THT:R_Axial_DIN0207_L6.3mm_D2.5mm_P2.54mm_Vertical, F.Cu at (184.3, 37.1)
- added R86: R_Axial_DIN0207_L6.3mm_D2.5mm_P2.54mm_Vertical, Resistor_THT:R_Axial_DIN0207_L6.3mm_D2.5mm_P2.54mm_Vertical, F.Cu at (178.9, 63.4)
- R57: value Potentiometer_Bourns_3266Y_Vertical -> 10K
- R58: value Potentiometer_Bourns_3266Y_Vertical -> 5K
- U41: value DIP-24_W15.24mm_LongPads -> CHR ROM
- U70: value DIP-14_W7.62mm_LongPads -> 7803
- U8: value DIP-40_W15.24mm_LongPads -> 6502
Routing:
- net (no net): track 62578.8 -> 62578.0 mm, vias 2261 -> 2211
Other:
- board text removed: "J2"
- board text removed: "J3"
- board text removed: "R38"
- board text removed: "R39"
- board text removed: "R40"
- board text removed: "R41"
- board text removed: "R42"
- board text removed: "R43"
- board text removed: "R44"
- board text removed: "R45"
- board text removed: "R46"
- board text removed: "R47"
- board text removed: "R48"
- board text removed: "R49"
- board text removed: "R86"
